File: Hardware/PSU Eurorack simple switched/PSU Eurorack simple switched.kicad_pcb (KiCad board)
At the start: 2 copper layers, 100 x 50 mm, 30 parts, among them J1 PWR_in, J2 PWR, J3 PWR, J4 CV_GATE, J5 PWR_out_1, J6 PWR_out_2, J7 PWR_out_3, U1 TDK CCG30-48-12D, U2 AMSR-78xx

Commit message: Swapped polarity of -12V LED, added remote control header, enlarged input area, fixed text placements
Parts:
- added J8: REMOTE, Connector_PinHeader_2.54mm:PinHeader_2x01_P2.54mm_Vertical, F.Cu at (82.5, 81.0)
- moved D3 2.64 mm to (134.8, 56.5), turned to 90 degrees
Connections:
- D3 pad 1: GND -> Net-(D3-Pad1)
- D3 pad 2: Net-(D3-Pad2) -> GND
- R4 pad 2: Net-(D3-Pad2) -> Net-(D3-Pad1)
- U1 pad 6: unconnected-(U1-Pad6) -> RC
Routing:
- net RC: track 0.00 -> 28.9 mm
- net Net-(D3-Pad2): track 2.55 -> 0.00 mm
- net Net-(D3-Pad1): track 0.00 -> 2.45 mm
Other:
- board text added: "© Fredrik Viklund February 2022"
- board text removed: "© Fredrik Viklund 14 Jan 2022"
