File: Hardware/PSU Eurorack simple switched/PSU Eurorack simple switched.kicad_sch (KiCad schematic)
At the start: 30 parts, among them J1 PWR_in, J2 PWR, J3 PWR, J4 CV_GATE, J5 PWR_out_1, J6 PWR_out_2, J7 PWR_out_3, U1 TDK CCG30-48-12D, U2 AMSR-78xx

Commit message: Swapped polarity of -12V LED, added remote control header, enlarged input area, fixed text placements
Parts:
- added J8: REMOTE, Connector_PinHeader_2.54mm:PinHeader_2x01_P2.54mm_Vertical, symbol Connector_Generic:Conn_01x02
- U1: symbol Fredriks:DKMW30 -> Fredriks:TDK_CCG30
Connections:
- net GND: now also D3.2 (A), J8.2 (Pin_2); no longer D3.1 (K)
- net at R4.2: now also D3.1 (K); no longer D3.2 (A)
- net RC: now reaches U1.6 (R.C.)
- net RC: now also J8.1 (Pin_1)
Other:
- moved on the sheet: D3, J2, J3

Commit message: Bus board first version with gerbers
Parts:
- added F1: 7 or 8A polyfuse, Fuse:Fuse_Bourns_MF-RG900, symbol Device:Polyfuse
Connections:
- net GND: now also D2.2 (A)
- net Vin: now also F1.1; no longer D2.2 (A), R1.2
- net at C1.1, D2.1 (K), U1.1 (Vin+)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: now also R1.2, F1.2
Other:
- moved on the sheet: C1, C2, D1, D2, D3, D4, D5, R1, R2, R3, R4, U1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
